Commit message: added ros2 files

File: husky_description/urdf/accessories/intel_realsense.urdf.xacro (robot description, xacro)
@@ -33,6 +33,5 @@
               <width>${width}</width>
               <height>${height}</height>
-              <!-- TODO: check what format the Realsense hardware delivers and set this to match! -->
-              <format>RGB_INT8</format>
+              <format>RGB8</format>
             </image>
             <clip>

File: husky_description/urdf/accessories/sensor_arch.urdf.xacro (robot description, xacro)
@@ -2,5 +2,4 @@
 <robot xmlns:xacro="http://ros.org/wiki/xacro" name="510_mm_sensor_arch">
     <xacro:macro name="sensor_arch" params="prefix parent size:=510 *origin">
-        <link name="${prefix}sensor_arch_base_link" />
         <!-- Spawn the sensor arch link -->
         <link name="${prefix}sensor_arch_mount_link">
@@ -18,14 +17,9 @@
              </collision>
         </link>
-        <joint name="${prefix}sensor_arch_base_link_joint" type="fixed">
-            <parent link="${parent}" />
-            <child link="${prefix}sensor_arch_base_link" />
-            <xacro:insert_block name="origin" />
-        </joint>
         <!-- Attach the sensor arch to the top plate -->
         <joint name="${prefix}sensor_arch_mount" type="fixed">
-             <parent link="${prefix}sensor_arch_base_link"/>
+             <xacro:insert_block name="origin"/>
+             <parent link="${parent}"/>
              <child link="${prefix}sensor_arch_mount_link"/>
-             <origin xyz="0 0 ${size/1000}" rpy="0 0 0" />
         </joint>
     </xacro:macro>

File: husky_description/urdf/decorations.urdf.xacro (robot description, xacro)
@@ -1,24 +1,3 @@
 <?xml version="1.0"?>
-<!--
-Software License Agreement (BSD)
-\file      decorations.urdf.xacro
-\authors   Paul Bovbel <pbovbel@clearpathrobotics.com>, Devon Ash <dash@clearpathrobotics.com>
-\copyright Copyright (c) 2015, Clearpath Robotics, Inc., All rights reserved.
-Redistribution and use in source and binary forms, with or without modification, are permitted provided that
-the following conditions are met:
- * Redistributions of source code must retain the above copyright notice, this list of conditions and the
-   following disclaimer.
- * Redistributions in binary form must reproduce the above copyright notice, this list of conditions and the
-   following disclaimer in the documentation and/or other materials provided with the distribution.
- * Neither the name of Clearpath Robotics nor the names of its contributors may be used to endorse or promote
-   products derived from this software without specific prior written permission.
-THIS SOFTWARE IS PROVIDED BY THE COPYRIGHT HOLDERS AND CONTRIBUTORS "AS IS" AND ANY EXPRESS OR IMPLIED WAR-
-RANTIES, INCLUDING, BUT NOT LIMITED TO, THE IMPLIED WARRANTIES OF MERCHANTABILITY AND FITNESS FOR A PARTICULAR
-PURPOSE ARE DISCLAIMED. IN NO EVENT SHALL THE COPYRIGHT HOLDER OR CONTRIBUTORS BE LIABLE FOR ANY DIRECT, IN-
-DIRECT, INCIDENTAL, SPECIAL, EXEMPLARY, OR CONSEQUENTIAL DAMAGES (INCLUDING, BUT NOT LIMITED TO, PROCUREMENT
-OF SUBSTITUTE GOODS OR SERVICES; LOSS OF USE, DATA, OR PROFITS; OR BUSINESS INTERRUPTION) HOWEVER CAUSED AND
-ON ANY THEORY OF LIABILITY, WHETHER IN CONTRACT, STRICT LIABILITY, OR TORT (INCLUDING NEGLIGENCE OR OTHERWISE)
-ARISING IN ANY WAY OUT OF THE USE OF THIS SOFTWARE, EVEN IF ADVISED OF THE POSSIBILITY OF SUCH DAMAGE.
--->
 <robot name="husky_decorations" xmlns:xacro="http://ros.org/wiki/xacro">
   <material name="dark_grey"><color rgba="0.2 0.2 0.2 1.0" /></material>
@@ -30,9 +9,6 @@
   <material name="red"><color rgba="1.0 0.0 0.0 1.0" /></material>
   <xacro:macro name="husky_decorate">
-    <xacro:property name="husky_front_bumper_enable"    value="$(optenv HUSKY_FRONT_BUMPER 1)" />
-    <xacro:property name="husky_rear_bumper_enable"     value="$(optenv HUSKY_REAR_BUMPER 1)" />
-    <xacro:property name="husky_front_bumper_extend"    value="$(optenv HUSKY_FRONT_BUMPER_EXTEND 0)" />
-    <xacro:property name="husky_rear_bumper_extend"     value="$(optenv HUSKY_REAR_BUMPER_EXTEND 0)" />
-    <xacro:property name="husky_wibotic_bumper_enable"  value="$(optenv HUSKY_WIBOTIC_BUMPER 0)" />
+    <xacro:property name="husky_front_bumper_extend" value="$(optenv HUSKY_FRONT_BUMPER_EXTEND 0)" />
+    <xacro:property name="husky_rear_bumper_extend" value="$(optenv HUSKY_REAR_BUMPER_EXTEND 0)" />
     <!-- Spawn Husky chassis -->
     <link name="top_chassis_link">
@@ -66,74 +42,58 @@
     </xacro:if>
     <!-- Spawn front bumper link -->
-    <xacro:if value="${husky_front_bumper_enable}">
-      <xacro:unless value="${husky_wibotic_bumper_enable}">
-        <link name="front_bumper_link">
+    <link name="front_bumper_link">
+      <visual>
+        <geometry>
+          <mesh filename="package://husky_description/meshes/bumper.dae" />
+        </geometry>
+      </visual>
+    </link>
+    <!-- Attach front bumper -->
+    <joint name="front_bumper" type="fixed">
+      <origin xyz="${0.48 + husky_front_bumper_extend} 0 0.091" rpy="0 0 0" />
+      <parent link="base_link" />
+      <child link="front_bumper_link" />
+    </joint>
+    <xacro:if value="${husky_front_bumper_extend}">
+      <link name="front_bumper_extension_link">
           <visual>
-            <geometry>
-              <mesh filename="package://husky_description/meshes/bumper.dae" />
-            </geometry>
+              <geometry>
+                  <mesh filename="package://husky_description/meshes/bumper_extension.dae" />
+              </geometry>
           </visual>
-        </link>
-      </xacro:unless>
-      <xacro:if value="${husky_wibotic_bumper_enable}">
-        <link name="front_bumper_link">
-          <visual>
-            <material name="black"/>
-            <geometry>
-              <mesh filename="package://husky_description/meshes/accessories/wibotic_bumper.stl" />
-            </geometry>
-          </visual>
-        </link>
-      </xacro:if>
-      <!-- Attach front bumper -->
-      <joint name="front_bumper" type="fixed">
+      </link>
+      <joint name="front_bumper_extension" type="fixed">
         <origin xyz="${0.48 + husky_front_bumper_extend} 0 0.091" rpy="0 0 0" />
         <parent link="base_link" />
-        <child link="front_bumper_link" />
+        <child link="front_bumper_extension_link" />
       </joint>
-      <xacro:if value="${husky_front_bumper_extend}">
-        <link name="front_bumper_extension_link">
-            <visual>
-                <geometry>
-                    <mesh filename="package://husky_description/meshes/bumper_extension.dae" />
-                </geometry>
-            </visual>
-        </link>
-        <joint name="front_bumper_extension" type="fixed">
-          <origin xyz="${0.48 + husky_front_bumper_extend} 0 0.091" rpy="0 0 0" />
-          <parent link="base_link" />
-          <child link="front_bumper_extension_link" />
-        </joint>
-      </xacro:if>
     </xacro:if>
     <!-- Spawn rear bumper link -->
-    <xacro:if value="${husky_rear_bumper_enable}">
-      <link name="rear_bumper_link">
-        <visual>
-          <geometry>
-            <mesh filename="package://husky_description/meshes/bumper.dae" />
-          </geometry>
-        </visual>
+    <link name="rear_bumper_link">
+      <visual>
+        <geometry>
+          <mesh filename="package://husky_description/meshes/bumper.dae" />
+        </geometry>
+      </visual>
+    </link>
+    <!-- Attach rear bumper -->
+    <joint name="rear_bumper" type="fixed">
+      <origin xyz="${-0.48 - husky_rear_bumper_extend} 0 0.091" rpy="0 0 ${M_PI}" />
+      <parent link="base_link" />
+      <child link="rear_bumper_link" />
+    </joint>
+    <xacro:if value="${husky_rear_bumper_extend}">
+      <link name="rear_bumper_extension_link">
+          <visual>
+              <geometry>
+                  <mesh filename="package://husky_description/meshes/bumper_extension.dae" />
+              </geometry>
+          </visual>
       </link>
-      <!-- Attach rear bumper -->
-      <joint name="rear_bumper" type="fixed">
+      <joint name="rear_bumper_extension" type="fixed">
         <origin xyz="${-0.48 - husky_rear_bumper_extend} 0 0.091" rpy="0 0 ${M_PI}" />
         <parent link="base_link" />
-        <child link="rear_bumper_link" />
+        <child link="rear_bumper_extension_link" />
       </joint>
-      <xacro:if value="${husky_rear_bumper_extend}">
-        <link name="rear_bumper_extension_link">
-            <visual>
-                <geometry>
-                    <mesh filename="package://husky_description/meshes/bumper_extension.dae" />
-                </geometry>
-            </visual>
-        </link>
-        <joint name="rear_bumper_extension" type="fixed">
-          <origin xyz="${-0.48 - husky_rear_bumper_extend} 0 0.091" rpy="0 0 ${M_PI}" />
-          <parent link="base_link" />
-          <child link="rear_bumper_extension_link" />
-        </joint>
-      </xacro:if>
     </xacro:if>
     <xacro:if value="$(optenv HUSKY_TOP_PLATE_ENABLED true)">
